Commit message: commit

File: urdf/rs_go.xacro (robot description, xacro)
@@ -1,7 +1,7 @@
 <?xml version="1.0" ?>
 <robot name="rs_go" xmlns:xacro="http://www.ros.org/wiki/xacro">
-<xacro:include filename="$(find rs_go_description)/urdf/materials.xacro" />
-<xacro:include filename="$(find rs_go_description)/urdf/rs_go.trans" />
-<xacro:include filename="$(find rs_go_description)/urdf/rs_go.gazebo" />
+<xacro:include filename="$(find rs_go)/urdf/materials.xacro" />
+<xacro:include filename="$(find rs_go)/urdf/rs_go.trans" />
+<xacro:include filename="$(find rs_go)/urdf/rs_go.gazebo" />
 <link name="base_link">
   <inertial>
@@ -13,5 +13,5 @@
     <origin rpy="0 0 0" xyz="0 0 0"/>
     <geometry>
-      <mesh filename="package://rs_go_description/meshes/base_link.stl" scale="0.001 0.001 0.001"/>
+      <mesh filename="package://rs_go/meshes/base_link.stl" scale="0.001 0.001 0.001"/>
     </geometry>
     <material name="rs_color"/>
@@ -20,5 +20,5 @@
     <origin rpy="0 0 0" xyz="0 0 0"/>
     <geometry>
-      <mesh filename="package://rs_go_description/meshes/base_link.stl" scale="0.001 0.001 0.001"/>
+      <mesh filename="package://rs_go/meshes/base_link.stl" scale="0.001 0.001 0.001"/>
     </geometry>
   </collision>
@@ -33,5 +33,5 @@
     <origin rpy="0 0 0" xyz="-0.0 -0.1 -0.05"/>
     <geometry>
-      <mesh filename="package://rs_go_description/meshes/front_left_wheel_1.stl" scale="0.001 0.001 0.001"/>
+      <mesh filename="package://rs_go/meshes/front_left_wheel_1.stl" scale="0.001 0.001 0.001"/>
     </geometry>
     <material name="black"/>
@@ -40,5 +40,5 @@
     <origin rpy="0 0 0" xyz="-0.0 -0.1 -0.05"/>
     <geometry>
-      <mesh filename="package://rs_go_description/meshes/front_left_wheel_1.stl" scale="0.001 0.001 0.001"/>
+      <mesh filename="package://rs_go/meshes/front_left_wheel_1.stl" scale="0.001 0.001 0.001"/>
     </geometry>
   </collision>
@@ -53,5 +53,5 @@
     <origin rpy="0 0 0" xyz="-0.0 -0.4 -0.05"/>
     <geometry>
-      <mesh filename="package://rs_go_description/meshes/back_left_wheel_1.stl" scale="0.001 0.001 0.001"/>
+      <mesh filename="package://rs_go/meshes/back_left_wheel_1.stl" scale="0.001 0.001 0.001"/>
     </geometry>
     <material name="black"/>
@@ -60,5 +60,5 @@
     <origin rpy="0 0 0" xyz="-0.0 -0.4 -0.05"/>
     <geometry>
-      <mesh filename="package://rs_go_description/meshes/back_left_wheel_1.stl" scale="0.001 0.001 0.001"/>
+      <mesh filename="package://rs_go/meshes/back_left_wheel_1.stl" scale="0.001 0.001 0.001"/>
     </geometry>
   </collision>
@@ -73,5 +73,5 @@
     <origin rpy="0 0 0" xyz="0.25 -0.1 -0.05"/>
     <geometry>
-      <mesh filename="package://rs_go_description/meshes/front_right_wheel_1.stl" scale="0.001 0.001 0.001"/>
+      <mesh filename="package://rs_go/meshes/front_right_wheel_1.stl" scale="0.001 0.001 0.001"/>
     </geometry>
     <material name="black"/>
@@ -80,5 +80,5 @@
     <origin rpy="0 0 0" xyz="0.25 -0.1 -0.05"/>
     <geometry>
-      <mesh filename="package://rs_go_description/meshes/front_right_wheel_1.stl" scale="0.001 0.001 0.001"/>
+      <mesh filename="package://rs_go/meshes/front_right_wheel_1.stl" scale="0.001 0.001 0.001"/>
     </geometry>
   </collision>
@@ -93,5 +93,5 @@
     <origin rpy="0 0 0" xyz="0.25 -0.4 -0.05"/>
     <geometry>
-      <mesh filename="package://rs_go_description/meshes/back_right_wheel_1.stl" scale="0.001 0.001 0.001"/>
+      <mesh filename="package://rs_go/meshes/back_right_wheel_1.stl" scale="0.001 0.001 0.001"/>
     </geometry>
     <material name="black"/>
@@ -100,5 +100,5 @@
     <origin rpy="0 0 0" xyz="0.25 -0.4 -0.05"/>
     <geometry>
-      <mesh filename="package://rs_go_description/meshes/back_right_wheel_1.stl" scale="0.001 0.001 0.001"/>
+      <mesh filename="package://rs_go/meshes/back_right_wheel_1.stl" scale="0.001 0.001 0.001"/>
     </geometry>
   </collision>

Commit message: obstacle avoidance feature added

File: urdf/rs_go.xacro (robot description, xacro)
@@ -151,5 +151,5 @@
 </joint>
 <joint name="sensor_laser_joint" type="fixed">
-  <origin xyz="-0.125 0.15 0.30" rpy="0.0 0.0 0.0"/>
+  <origin xyz="-0.125 0.15 0.30" rpy="0.0 0.0 -1.570796"/>
   <parent link="base_link"/>
   <child link="sensor_laser"/>
